File: pcb/HANmodule.sch (KiCad schematic (older format))
At the start: 32 parts, among them J1 HAN port, J2 Debug, J3 Prog, SW1 Reset, U1 RT9013-3.3v, U2 ESP-12F

Commit message: Updated schematic
Parts:
- removed C2: CP, Capacitor_THT:CP_Radial_D10.0mm_P5.00mm, symbol Device:CP_Small
- added C2: 100n, Capacitor_SMD:C_0603_1608Metric_Pad1.05x0.95mm_HandSolder, symbol Device:C_Small
- added U3: MAX6380-4v, symbol Power_Supervisor:TCM809
- C1: value CP -> 1F 5.5V; footprint Capacitor_THT:CP_Radial_D10.0mm_P5.00mm -> Capacitor_THT:CP_Radial_D22.0mm_P10.00mm_SnapIn
- R8: value 10k -> 100k
- U1: symbol dk_PMIC-Voltage-Regulators-Linear:MIC5219-3_3YM5-TR -> HANmodule-rescue:MIC5219-3_3YM5-TR-dk_PMIC-Voltage-Regulators-Linear
Connections:
- net labels added: +4V, RX, TX
- net labels removed: RST
- wire segments 80 -> 96
Other:
- note added: "DTR"
- note added: "GND"
- note added: "RTS"
- note added: "RX"
- note added: "TX"
- note added: "VCC"
- moved on the sheet: C1

Commit message: PCB rev 1
Parts:
- removed C1: 1F 5.5V, Capacitor_THT:CP_Radial_D22.0mm_P10.00mm_SnapIn, symbol Device:CP_Small
- removed C2: 100n, Capacitor_SMD:C_0603_1608Metric_Pad1.05x0.95mm_HandSolder, symbol Device:C_Small
- removed D1: D_Schottky, Diode_SMD:D_SMA-SMB_Universal_Handsoldering, symbol Device:D_Schottky
- removed D3: Meter data, LED_THT:LED_D3.0mm, symbol Device:LED
- removed D4: Wifi, LED_THT:LED_D3.0mm, symbol Device:LED
- removed D5: MQTT, LED_THT:LED_D3.0mm, symbol Device:LED
- removed R3, R8: 100k, Resistor_SMD:R_0603_1608Metric_Pad1.05x0.95mm_HandSolder, symbol Device:R_Small
- removed R4, R5: 1k, Resistor_SMD:R_0603_1608Metric_Pad1.05x0.95mm_HandSolder, symbol Device:R
- removed U1: RT9013-3.3v, Package_TO_SOT_SMD:SOT-23-5_HandSoldering, symbol HANmodule-rescue:MIC5219-3_3YM5-TR-dk_PMIC-Voltage-Regulators-Linear
- removed U3: MAX6380-4v, symbol Power_Supervisor:TCM809
- added C2: 0.1F 5.5V FC0H104ZFTBR24, Capacitor_SMD:CP_Elec_10x10.5, symbol Device:CP
- added C4: 1n, Capacitor_SMD:C_0603_1608Metric_Pad1.05x0.95mm_HandSolder, symbol Device:C_Small
- added C5: 100n, Capacitor_SMD:C_0603_1608Metric_Pad1.05x0.95mm_HandSolder, symbol Device:C_Small
- added C6: 1,75u, Capacitor_SMD:C_0603_1608Metric_Pad1.05x0.95mm_HandSolder, symbol Device:C_Small
- added Q1: SI2301DS_P-FET, Package_TO_SOT_SMD:SOT-23_Handsoldering, symbol Discrete:SI2301DS_P-FET
- added Q2: BSS139, Package_TO_SOT_SMD:SOT-23_Handsoldering, symbol Transistor_FET:BSS138
- added R11: 10k, Resistor_SMD:R_0603_1608Metric_Pad1.05x0.95mm_HandSolder, symbol Device:R_Small
- added R13: 102k, Resistor_SMD:R_0603_1608Metric_Pad1.05x0.95mm_HandSolder, symbol Device:R_Small
- added R14: 34k, Resistor_SMD:R_0603_1608Metric_Pad1.05x0.95mm_HandSolder, symbol Device:R_Small
- added R5: 113k, Resistor_SMD:R_0603_1608Metric_Pad1.05x0.95mm_HandSolder, symbol Device:R_Small
- added R6: 13k3, Resistor_SMD:R_0603_1608Metric_Pad1.05x0.95mm_HandSolder, symbol Device:R_Small
- added U1: TLV75530PDBV | RT9013, Package_TO_SOT_SMD:SOT-23-5_HandSoldering, symbol Regulator_Linear:TLV75530PDBV
- added U2: NCP308SNADJT1G, Package_SO:TSOP-6_1.65x3.05mm_P0.95mm, symbol IC:NCV308
- D1: renamed from D2; footprint LED_THT:LED_D3.0mm -> LED_SMD:LED_0805_2012Metric_Pad1.15x1.40mm_HandSolder
- D2: renamed from D6; footprint LED_THT:LED_D3.0mm -> LED_SMD:LED_0805_2012Metric_Pad1.15x1.40mm_HandSolder
- J1: value HAN port -> M20-7920342R; footprint Connector_PinSocket_2.54mm:PinSocket_2x03_P2.54mm_Horizontal -> SamacSys_Parts:M20-7920342R; symbol Connector_Generic:Conn_02x03_Counter_Clockwise -> Connector_Generic:Conn_02x03_Odd_Even
- J2: footprint Connector_PinHeader_2.54mm:PinHeader_1x02_P2.54mm_Vertical -> Connector_PinHeader_2.54mm:PinHeader_1x02_P2.54mm_Horizontal
- J3: footprint Connector_PinSocket_2.54mm:PinSocket_1x06_P2.54mm_Vertical -> Connector_PinHeader_2.54mm:PinHeader_1x06_P2.54mm_Horizontal
- R12: value 1k -> 100k
- R15: renamed from R13; value 1k -> 100k
- R2: value 1k -> 55R
- SW1: footprint Button_Switch_SMD:Panasonic_EVQPUJ_EVQPUA -> Button_Switch_SMD:Panasonic_EVQPUM_EVQPUD
- renumbered C3 to C1, C4 to C3, C5 to C7, C6 to C8, C7 to C9, R11 to R10, R6 to R4, R9 to R8, R10 to R9, U2 to U3
Connections:
- net +4V: now also R2.1, C2.1, C5.2, Q2.2 (S), R13.2, R5.1, U1.1 (IN), U1.3 (EN), U2.6 (VCC)
- net DIN: now also J1.3 (Pin_3); no longer J1.2 (Pin_2), R15.1
- net DOUT: now also J1.4 (Pin_4), R15.1; no longer J1.5 (Pin_5)
- net EN: now also Q2.1 (G), R11.2, U2.1 (~Reset)
- net GND: now also J1.6 (Pin_6), C2.2, C4.2, C5.1, C6.2, Q1.1 (G), R14.1, R6.2, U1.2 (GND), U2.2 (GND); no longer J1.4 (Pin_4)
- net GPIO0: no longer D1.1 (K)
- net VCC: now also J1.5 (Pin_5), Q1.3 (D); no longer J1.3 (Pin_3)
- net ~RST: now also U3.4 (GPIO16)
- net at R2.2: now also Q1.2 (S), Q2.3 (D)
- net at U3.2 (ADC): now also R13.1, R14.2
- net +3V3 renamed +3V0
- net +3V0: now also R11.1, U1.5 (OUT); no longer R2.1
- net FAULT_LED: no longer names the net of U3.5 (GPIO14)
- net FAULT_LED: no longer D2.1 (K)
- net MD_LED renamed ~LED
- net ~LED: now also D1.1 (K)
- net MQTT_LED: no longer names the net of U3.6 (GPIO12)
- net WIFI_LED renamed ~FAULT_LED
- net ~FAULT_LED: now also D2.1 (K)
- new net: C6.1, U2.4 (CT)
- new net: C4.1, R5.2, R6.1, U2.5 (Sense)
- no-connect marks 13 -> 15
Other:
- note added: "0.405v"
- note added: "3.846V\nThreshold"
- note added: "3V LDO"
- note added: "75mA @ 4.15V"
- note added: "depl. mode"
- moved on the sheet: C1, C3, C7, C8, C9, D1, D2, J1, J2, J3, R1, R10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

Commit message: PCB rev2 to be tested
Parts:
- removed Q2: BSS139, Package_TO_SOT_SMD:SOT-23_Handsoldering, symbol Transistor_FET:BSS138
- removed R2: 55R, Resistor_SMD:R_0603_1608Metric_Pad1.05x0.95mm_HandSolder, symbol Device:R
- removed U1: TLV75530PDBV | RT9013, Package_TO_SOT_SMD:SOT-23-5_HandSoldering, symbol Regulator_Linear:TLV75530PDBV
- added L1: 2.2UH 4x4mm, Inductor_SMD:L_Bourns-SRN4018, symbol Device:L_Small
- added Q2: BC807, Package_TO_SOT_SMD:SOT-23, symbol Transistor_BJT:BC807
- added R16: 1k, Resistor_SMD:R_0603_1608Metric_Pad1.05x0.95mm_HandSolder, symbol Device:R_Small
- added R17: 2k7, Resistor_SMD:R_0603_1608Metric_Pad1.05x0.95mm_HandSolder, symbol Device:R_Small
- added R18: 330k, Resistor_SMD:R_0603_1608Metric_Pad1.05x0.95mm_HandSolder, symbol Device:R_Small
- added R19: 100k, Resistor_SMD:R_0603_1608Metric_Pad1.05x0.95mm_HandSolder, symbol Device:R_Small
- added R2: 4k7, Resistor_SMD:R_0603_1608Metric_Pad1.05x0.95mm_HandSolder, symbol Device:R_Small
- added R20: 100k, Resistor_SMD:R_0603_1608Metric_Pad1.05x0.95mm_HandSolder, symbol Device:R
- added R3: NC, Resistor_SMD:R_0603_1608Metric_Pad1.05x0.95mm_HandSolder, symbol Device:R_Small
- added U1: TLV62568DBV, Package_TO_SOT_SMD:SOT-23-5, symbol Regulator_Switching:TLV62568DBV
- C1: value 1uF -> 4.7uF
- C3: value 1uF -> 10uF
- Q1: footprint Package_TO_SOT_SMD:SOT-23_Handsoldering -> Package_TO_SOT_SMD:SOT-23
Connections:
- net +3V0: now also L1.2, R18.1
- net +4V: now also Q2.3 (C), U1.1 (EN), U1.4 (VIN)
- net DIN: now also R20.1
- net GND: now also R17.1, R19.2, U1.2 (GND)
- net GPIO15: now also R20.2
- net at Q1.2 (S): now also R16.2, R2.2, R3.2
- new net: Q2.2 (E), R2.1, R3.1
- new net: Q2.1 (B), R16.1, R17.2
- new net: L1.1, U1.3 (SW)
- new net: R18.2, R19.1, U1.5 (FB)
- no-connect marks 15 -> 13
Other:
- note added: "2.58V"
- note removed: "75mA @ 4.15V"
- note removed: "depl. mode"
- moved on the sheet: C2, C3, C4, C5, C6, R11, R5, R6, U2

Commit message: Improved power design
Parts:
- removed Q2: BC807, Package_TO_SOT_SMD:SOT-23, symbol Transistor_BJT:BC807
- added D3, D4: LL4148, Diode_SMD:D_MiniMELF, symbol Device:D_Small
- added Q2: SI2301DS_P-FET, Package_TO_SOT_SMD:SOT-23, symbol HANmodule-rescue:SI2301DS_P-FET-Discrete
- added Q3: SI2302DS/2N7002, Package_TO_SOT_SMD:SOT-23, symbol Discrete:SI2302DS_N-FET
- added R21: 0R, Resistor_SMD:R_0603_1608Metric_Pad1.05x0.95mm_HandSolder, symbol Device:R_Small
- added R22: NC, Resistor_SMD:R_0603_1608Metric_Pad1.05x0.95mm_HandSolder, symbol Device:R_Small
- C1: footprint Capacitor_SMD:C_0603_1608Metric_Pad1.05x0.95mm_HandSolder -> Capacitor_SMD:C_0603_1608Metric
- C2: value 0.1F 5.5V FC0H104ZFTBR24 -> 0.47F; footprint Capacitor_SMD:CP_Elec_10x10.5 -> housings:c_sup 17,3x15x8.5P12
- C6: value 1,75u -> 1.5u
- D1, D2: footprint LED_SMD:LED_0805_2012Metric_Pad1.15x1.40mm_HandSolder -> LED_SMD:LED_0603_1608Metric
- Q1: symbol Discrete:SI2301DS_P-FET -> HANmodule-rescue:SI2301DS_P-FET-Discrete
- R13: value 102k -> 100k
- R14: value 34k -> 33k
- R16: value 1k -> 10k
- R17: value 2k7 -> 4k3
- R2: value 4k7 -> 4R7
- R3: value NC -> 5R6
- R5: value 113k -> 110k
- R6: value 13k3 -> 16k
- U2: symbol IC:NCV308 -> HANmodule-rescue:NCV308-IC
Connections:
- net +4V: now also Q2.3 (D)
- net EN: now also Q3.1 (G)
- net GND: now also Q3.2 (S)
- net at Q1.2 (S), R2.2, R3.2: now also R21.2; no longer R16.2
- net at R2.1, R3.1: now also Q2.2 (S)
- net at R16.1, R17.2: now also D4.1 (K), R22.2
- new net: Q2.1 (G), Q3.3 (D), R16.2
- new net: D3.1 (K), D4.2 (A), R22.1
- new net: D3.2 (A), R21.1
Other:
- note added: "1.18v drop"
- note added: "3.19V\nThreshold"
- note added: "3.87v"
- note removed: "3.846V\nThreshold"
- moved on the sheet: R16, R17
Changed lines of the file:
@@
 F 0 "D1" V 2139 5858 50  0000 R CNN
 F 1 "Heartbeat" V 2050 6425 50  0000 R CNN
-F 2 "LED_SMD:LED_0805_2012Metric_Pad1.15x1.40mm_HandSolder" H 2100 5975 50  0001 C CNN
+F 2 "LED_SMD:LED_0603_1608Metric" H 2100 5975 50  0001 C CNN
 F 3 "~" H 2100 5975 50  0001 C CNN
 	1    2100 5975
@@
 F 0 "D2" V 2489 5858 50  0000 R CNN
 F 1 "Fault" V 2398 5858 50  0000 R CNN
-F 2 "LED_SMD:LED_0805_2012Metric_Pad1.15x1.40mm_HandSolder" H 2450 5975 50  0001 C CNN
+F 2 "LED_SMD:LED_0603_1608Metric" H 2450 5975 50  0001 C CNN
 F 3 "~" H 2450 5975 50  0001 C CNN
 	1    2450 5975
@@
 P 5950 3825
 F 0 "R13" V 5754 3825 50  0000 C CNN
-F 1 "102k" V 5845 3825 50  0000 C CNN
+F 1 "100k" V 5845 3825 50  0000 C CNN
 F 2 "Resistor_SMD:R_0603_1608Metric_Pad1.05x0.95mm_HandSolder" H 5950 3825 50  0001 C CNN
 F 3 "~" H 5950 3825 50  0001 C CNN
@@
 P 5950 4100
 F 0 "R14" V 5754 4100 50  0000 C CNN
-F 1 "34k" V 5845 4100 50  0000 C CNN
+F 1 "33k" V 5845 4100 50  0000 C CNN
 F 2 "Resistor_SMD:R_0603_1608Metric_Pad1.05x0.95mm_HandSolder" H 5950 4100 50  0001 C CNN
 F 3 "~" H 5950 4100 50  0001 C CNN
@@
 F 0 "C1" H 1700 3300 50  0000 L CNN
 F 1 "4.7uF" H 1700 3175 50  0000 L CNN
-F 2 "Capacitor_SMD:C_0603_1608Metric_Pad1.05x0.95mm_HandSolder" H 1875 3250 50  0001 C CNN
+F 2 "Capacitor_SMD:C_0603_1608Metric" H 1875 3250 50  0001 C CNN
 F 3 "~" H 1875 3250 50  0001 C CNN
 	1    1875 3250
@@
 P 3575 1425
 F 0 "C2" H 3425 1325 50  0000 L CNN
-F 1 "0.1F 5.5V FC0H104ZFTBR24" V 3725 1025 50  0000 L CNN
-F 2 "Capacitor_SMD:CP_Elec_10x10.5" H 3613 1275 50  0001 C CNN
+F 1 "0.47F" V 3725 1350 50  0000 L CNN
+F 2 "housings:c_sup 17,3x15x8.5P12" H 3613 1275 50  0001 C CNN
 F 3 "~" H 3575 1425 50  0001 C CNN
 	1    3575 1425
@@
 P 4100 1525
 F 0 "R6" H 4159 1571 50  0000 L CNN
-F 1 "13k3" H 4159 1480 50  0000 L CNN
+F 1 "16k" H 4159 1480 50  0000 L CNN
 F 2 "Resistor_SMD:R_0603_1608Metric_Pad1.05x0.95mm_HandSolder" H 4100 1525 50  0001 C CNN
 F 3 "~" H 4100 1525 50  0001 C CNN
@@
 P 4100 1325
 F 0 "R5" H 4159 1371 50  0000 L CNN
-F 1 "113k" H 4159 1280 50  0000 L CNN
+F 1 "110k" H 4159 1280 50  0000 L CNN
 F 2 "Resistor_SMD:R_0603_1608Metric_Pad1.05x0.95mm_HandSolder" H 4100 1325 50  0001 C CNN
 F 3 "~" H 4100 1325 50  0001 C CNN
@@
 Wire Wire Line
 	4100 1700 4100 1625
-Connection ~ 3575 1700
 Wire Wire Line
 	3575 1150 4100 1150
@@
 	4100 1150 4100 1225
 Connection ~ 3575 1150
-Connection ~ 3450 1150
-$Comp
-L IC:NCV308 U2
+$Comp
+L HANmodule-rescue:NCV308-IC U2
 U 1 1 5E3DDDE0
 P 4950 1425
@@
 P 5450 1550
 F 0 "C6" H 5542 1596 50  0000 L CNN
-F 1 "1,75u" H 5475 1475 50  0000 L CNN
+F 1 "1.5u" H 5475 1475 50  0000 L CNN
 F 2 "Capacitor_SMD:C_0603_1608Metric_Pad1.05x0.95mm_HandSolder" H 5450 1550 50  0001 C CNN
 F 3 "~" H 5450 1550 50  0001 C CNN
@@
 	7625 4550 7825 4550
 $Comp
-L Discrete:SI2301DS_P-FET Q1
+L HANmodule-rescue:SI2301DS_P-FET-Discrete Q1
 U 1 1 5E3D975A
 P 1650 1250
@@
 0.405v
 Text Notes 3975 1075 0    50   ~ 0
-3.846V\nThreshold
+3.19V\nThreshold
 $Comp
 L power:+4V #PWR03
@@
 L power:GND #PWR0101
 U 1 1 5E42056B
-P 2500 1825
-F 0 "#PWR0101" H 2500 1575 50  0001 C CNN
-F 1 "GND" H 2505 1652 50  0000 C CNN
-F 2 "" H 2500 1825 50  0001 C CNN
-F 3 "" H 2500 1825 50  0001 C CNN
-	1    2500 1825
+P 2550 1975
+F 0 "#PWR0101" H 2550 1725 50  0001 C CNN
+F 1 "GND" H 2555 1802 50  0000 C CNN
+F 2 "" H 2550 1975 50  0001 C CNN
+F 3 "" H 2550 1975 50  0001 C CNN
+	1    2550 1975
 	1    0    0    -1
 $EndComp
@@
 L Device:R_Small R16
 U 1 1 5ED563C3
-P 2200 1475
-F 0 "R16" V 2275 1450 50  0000 C CNN
-F 1 "1k" V 2095 1475 50  0000 C CNN
-F 2 "Resistor_SMD:R_0603_1608Metric_Pad1.05x0.95mm_HandSolder" H 2200 1475 50  0001 C CNN
-F 3 "~" H 2200 1475 50  0001 C CNN
-	1    2200 1475
-	0    1    1    0
-$EndComp
-$Comp
-L Transistor_BJT:BC807 Q2
-U 1 1 5ED57471
-P 2500 1250
-F 0 "Q2" V 2828 1250 50  0000 C CNN
-F 1 "BC807" V 2737 1250 50  0000 C CNN
-F 2 "Package_TO_SOT_SMD:SOT-23" H 2700 1175 50  0001 L CIN
-F 3 "http://www.fairchildsemi.com/ds/BC/BC807.pdf" H 2500 1250 50  0001 L CNN
-	1    2500 1250
-	0    1    -1   0
+P 2550 1550
+F 0 "R16" H 2425 1500 50  0000 C CNN
+F 1 "10k" H 2425 1575 50  0000 C CNN
+F 2 "Resistor_SMD:R_0603_1608Metric_Pad1.05x0.95mm_HandSolder" H 2550 1550 50  0001 C CNN
+F 3 "~" H 2550 1550 50  0001 C CNN
+	1    2550 1550
+	-1   0    0    1
 $EndComp
 $Comp
 L Device:R_Small R17
 U 1 1 5ED59805
-P 2500 1600
-F 0 "R17" H 2441 1554 50  0000 R CNN
-F 1 "2k7" H 2441 1645 50  0000 R CNN
-F 2 "Resistor_SMD:R_0603_1608Metric_Pad1.05x0.95mm_HandSolder" H 2500 1600 50  0001 C CNN
-F 3 "~" H 2500 1600 50  0001 C CNN
-	1    2500 1600
+P 2550 1750
+F 0 "R17" H 2491 1704 50  0000 R CNN
+F 1 "4k3" H 2491 1795 50  0000 R CNN
+F 2 "Resistor_SMD:R_0603_1608Metric_Pad1.05x0.95mm_HandSolder" H 2550 1750 50  0001 C CNN
+F 3 "~" H 2550 1750 50  0001 C CNN
+	1    2550 1750
 	-1   0    0    1
 $EndComp
@@
 P 2150 1050
 F 0 "R2" V 2100 875 50  0000 C CNN
-F 1 "4k7" V 2045 1050 50  0000 C CNN
+F 1 "4R7" V 2045 1050 50  0000 C CNN
 F 2 "Resistor_SMD:R_0603_1608Metric_Pad1.05x0.95mm_HandSolder" H 2150 1050 50  0001 C CNN
 F 3 "~" H 2150 1050 50  0001 C CNN
@@
 $EndComp
 Wire Wire Line
-	1850 1150 2050 1150
+	1850 1150 1975 1150
 Connection ~ 2050 1150
 Wire Wire Line
 	2250 1150 2275 1150
 Wire Wire Line
-	2100 1475 2050 1475
-Wire Wire Line
-	2050 1475 2050 1150
-Wire Wire Line
-	2300 1475 2500 1475
-Wire Wire Line
-	2500 1475 2500 1450
-Wire Wire Line
 	2050 1050 2050 1150
 Wire Wire Line
-	2500 1500 2500 1475
-Connection ~ 2500 1475
-Wire Wire Line
-	2500 1700 2500 1825
-Wire Wire Line
-	2500 1700 3575 1700
-Connection ~ 2500 1700
+	2550 1850 2550 1975
 Wire Wire Line
 	5550 1325 5875 1325
-Wire Wire Line
-	2700 1150 3450 1150
 Wire Wire Line
 	2250 1050 2275 1050
@@
 	2275 1050 2275 1150
 Connection ~ 2275 1150
-Wire Wire Line
-	2275 1150 2300 1150
 $Comp
 L Device:R_Small R3
 U 1 1 5ED554DE
 P 2150 1150
-F 0 "R3" V 2225 975 50  0000 C CNN
-F 1 "NC" V 2225 1150 50  0000 C CNN
+F 0 "R3" V 2225 1275 50  0000 C CNN
+F 1 "5R6" V 2225 1150 50  0000 C CNN
 F 2 "Resistor_SMD:R_0603_1608Metric_Pad1.05x0.95mm_HandSolder" H 2150 1150 50  0001 C CNN
 F 3 "~" H 2150 1150 50  0001 C CNN
@@
 Wire Wire Line
 	850  1550 725  1550
+$Comp
+L HANmodule-rescue:SI2301DS_P-FET-Discrete Q2
+U 1 1 5F4E2EAA
+P 2600 1250
+F 0 "Q2" V 2905 1250 40  0000 C CNN
+F 1 "SI2301DS_P-FET" V 2829 1250 40  0000 C CNN
+F 2 "Package_TO_SOT_SMD:SOT-23" H 2470 1352 29  0001 C CNN
+F 3 "" H 2600 1250 60  0000 C CNN
+	1    2600 1250
+	0    1    -1   0
+$EndComp
+$Comp
+L Device:D_Small D3
+U 1 1 5F4ED3DC
+P 2125 1650
+F 0 "D3" H 2150 1575 50  0000 C CNN
+F 1 "LL4148" H 2225 1750 50  0000 C CNN
+F 2 "Diode_SMD:D_MiniMELF" V 2125 1650 50  0001 C CNN
+F 3 "~" V 2125 1650 50  0001 C CNN
+	1    2125 1650
+	-1   0    0    1
+$EndComp
+$Comp
+L Device:D_Small D4
+U 1 1 5F4EDE59
+P 2325 1650
+F 0 "D4" H 2350 1575 50  0000 C CNN
+F 1 "LL4148" H 2350 1750 50  0000 C CNN
+F 2 "Diode_SMD:D_MiniMELF" V 2325 1650 50  0001 C CNN
+F 3 "~" V 2325 1650 50  0001 C CNN
+	1    2325 1650
+	-1   0    0    1
+$EndComp
+Wire Wire Line
+	1975 1650 2025 1650
+Connection ~ 2550 1650
+Text Notes 2075 1850 0    50   ~ 0
+1.18v drop
+Text Notes 3150 1125 0    50   ~ 0
+3.87v
+Wire Wire Line
+	2275 1150 2400 1150
+$Comp
+L Discrete:SI2302DS_N-FET Q3
+U 1 1 5F529F9F
+P 3150 1775
+F 0 "Q3" H 3341 1813 40  0000 L CNN
+F 1 "SI2302DS/2N7002" H 2625 1600 40  0000 L CNN
+F 2 "Package_TO_SOT_SMD:SOT-23" H 3020 1877 29  0001 C CNN
+F 3 "" H 3150 1775 60  0000 C CNN
+	1    3150 1775
+	-1   0    0    -1
+$EndComp
+$Comp
+L power:GND #PWR024
+U 1 1 5F53B53D
+P 5350 1700
+F 0 "#PWR024" H 5350 1450 50  0001 C CNN
+F 1 "GND" H 5355 1527 50  0000 C CNN
+F 2 "" H 5350 1700 50  0001 C CNN
+F 3 "" H 5350 1700 50  0001 C CNN
+	1    5350 1700
+	1    0    0    -1
+$EndComp
+$Comp
+L power:GND #PWR023
+U 1 1 5F53BA71
+P 3050 1975
+F 0 "#PWR023" H 3050 1725 50  0001 C CNN
+F 1 "GND" H 3055 1802 50  0000 C CNN
+F 2 "" H 3050 1975 50  0001 C CNN
+F 3 "" H 3050 1975 50  0001 C CNN
+	1    3050 1975
+	1    0    0    -1
+$EndComp
+Wire Wire Line
+	2550 1450 3050 1450
+Connection ~ 2550 1450
+Wire Wire Line
+	3050 1450 3050 1575
+Text Label 3675 1825 2    50   ~ 0
+EN
+Wire Wire Line
+	3350 1825 3675 1825
+Wire Wire Line
+	3450 1150 2800 1150
+Connection ~ 3450 1150
+$Comp
+L Device:R_Small R21
+U 1 1 5F5896AB
+P 1975 1400
+F 0 "R21" H 2075 1375 50  0000 C CNN
+F 1 "0R" H 2075 1450 50  0000 C CNN
+F 2 "Resistor_SMD:R_0603_1608Metric_Pad1.05x0.95mm_HandSolder" H 1975 1400 50  0001 C CNN
+F 3 "~" H 1975 1400 50  0001 C CNN
+	1    1975 1400
+	-1   0    0    1
+$EndComp
+Wire Wire Line
+	1975 1500 1975 1650
+Wire Wire Line
+	1975 1300 1975 1150
+Connection ~ 1975 1150
+Wire Wire Line
+	1975 1150 2050 1150
+Wire Wire Line
+	2425 1650 2425 1500
+Wire Wire Line
+	2425 1650 2550 1650
+Connection ~ 2425 1650
+$Comp
+L Device:R_Small R22
+U 1 1 5F59079B
+P 2325 1500
+F 0 "R22" H 2425 1475 50  0000 C CNN
+F 1 "NC" H 2425 1550 50  0000 C CNN
+F 2 "Resistor_SMD:R_0603_1608Metric_Pad1.05x0.95mm_HandSolder" H 2325 1500 50  0001 C CNN
+F 3 "~" H 2325 1500 50  0001 C CNN
+	1    2325 1500
+	0    -1   -1   0
+$EndComp
+Wire Wire Line
+	2225 1500 2225 1650
+Connection ~ 2225 1650
 $EndSCHEMATC
